File: HL2_Companion.kicad_pcb (KiCad board)
At the start: 2 copper layers, 99.9 x 100 mm, 194 parts, among them CN7 CONN_01X02, J1 CONN_02X05, J33 SJ-43514-SMT, J34 SJ-43514-SMT, K1 EA2-NJ, K2 EA2-NJ, K3 EA2-NJ, K4 EA2-NJ, K5 EA2-NJ, K6 EA2-NJ, K7 EA2-NJ, P1 CONN_01X02, P2 FFC 20pin, P3 CONN_01X04, P4 CONN_01X04, P5 CONN_01X02, P6 CONN_01X06, P7 CONN_01X02, P8 CONN_01X02, Q1 2N27002, Q2 2N27002, Q3 2N27002, Q4 2N27002, Q5 DTC144E, Q50 SM05, Q51 SM05, Q6 IRLML6402, Q7 DTC144E, Q8 IRLML6402, Q9 DTC144E, T1 FAR-REV_Tran, U1 MCP23008-SSOP, U18 AK4951AEN, U2 AD8692ARZ, U20 TAR5SB33, U21 ST1S10, U22 PIC12F1822-E/SN, U3 74LVC1G04, U4 ULN2803A, U5 TPS730

Commit message: Gerber corrected
Routing:
- net (no net): track 14.5 -> 0.00 mm, vias 5 -> 0
Changed lines of the file:
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@@
     (thickness 1.6)
     (drawings 86)
-    (tracks 2476)
+    (tracks 2465)
     (zones 0)
     (modules 194)
@@
     (visible_elements 7FFEFF7F)
     (pcbplotparams
-      (layerselection 0x3f0ff_80000001)
+      (layerselection 0x030fc_80000001)
       (usegerberextensions false)
       (excludeedgelayer true)
@@
   (gr_line (start 169.95 40) (end 169.95 140) (angle 90) (layer Edge.Cuts) (width 0.15))
   (gr_line (start 70 40) (end 70 140) (angle 90) (layer Edge.Cuts) (width 0.15))
-  (segment (start 85.598 121.666) (end 85.598 123.952) (width 0.3) (layer B.Cu) (net 0))
-  (via (at 78.994 126.238) (size 0.6) (drill 0.3) (layers F.Cu B.Cu) (net 0))
-  (segment (start 78.994 126.238) (end 83.312 126.238) (width 0.3) (layer F.Cu) (net 0))
-  (via (at 83.312 126.238) (size 0.6) (drill 0.3) (layers F.Cu B.Cu) (net 0))
-  (segment (start 83.312 126.238) (end 85.598 123.952) (width 0.3) (layer B.Cu) (net 0))
-  (via (at 85.598 123.952) (size 0.6) (drill 0.3) (layers F.Cu B.Cu) (net 0))
-  (segment (start 78.994 126.238) (end 78.994 128.27) (width 0.3) (layer B.Cu) (net 0))
-  (via (at 85.598 121.666) (size 0.6) (drill 0.3) (layers F.Cu B.Cu) (net 0))
-  (segment (start 78.994 128.27) (end 78.994 128.778) (width 0.3) (layer B.Cu) (net 0))
-  (via (at 77.47 130.302) (size 0.6) (drill 0.3) (layers F.Cu B.Cu) (net 0))
-  (segment (start 78.994 128.778) (end 77.47 130.302) (width 0.3) (layer B.Cu) (net 0))
   (segment (start 163.55 96.13) (end 159.99 99.69) (width 1) (layer B.Cu) (net 1))
   (segment (start 159.238 100.352) (end 159.238 101.6) (width 1) (layer B.Cu) (net 1))
